Commit message: Fixed xacro math expressions

File: robot_specific_config/abb_irb120_support/urdf/irb120.ros2_control.xacro (robot description, xacro)
@@ -24,6 +24,6 @@
       <joint name="${prefix}joint_1">
         <command_interface name="position">
-          <param name="min">$(-165 * pi / 180)</param>
-          <param name="max">$(165 * pi / 180)</param>
+          <param name="min">${-165 * pi / 180}</param>
+          <param name="max">${165 * pi / 180}</param>
         </command_interface>
         <command_interface name="velocity"/>
@@ -35,6 +35,6 @@
       <joint name="${prefix}joint_2">
         <command_interface name="position">
-          <param name="min">$(-110 * pi / 180)</param>
-          <param name="max">$(110 * pi / 180)</param>
+          <param name="min">${-110 * pi / 180}</param>
+          <param name="max">${110 * pi / 180}</param>
         </command_interface>
         <command_interface name="velocity"/>
@@ -46,6 +46,6 @@
       <joint name="${prefix}joint_3">
         <command_interface name="position">
-          <param name="min">$(-110 * pi / 180)</param>
-          <param name="max">$(70 * pi / 180)</param>
+          <param name="min">${-110 * pi / 180}</param>
+          <param name="max">${70 * pi / 180}</param>
         </command_interface>
         <command_interface name="velocity"/>
@@ -57,6 +57,6 @@
       <joint name="${prefix}joint_4">
         <command_interface name="position">
-          <param name="min">$(-160 * pi / 180)</param>
-          <param name="max">$(160 * pi / 180)</param>
+          <param name="min">${-160 * pi / 180}</param>
+          <param name="max">${160 * pi / 180}</param>
         </command_interface>
         <command_interface name="velocity"/>
@@ -68,6 +68,6 @@
       <joint name="${prefix}joint_5">
         <command_interface name="position">
-          <param name="min">$(-120 * pi / 180)</param>
-          <param name="max">$(120 * pi / 180)</param>
+          <param name="min">${-120 * pi / 180}</param>
+          <param name="max">${120 * pi / 180}</param>
         </command_interface>
         <command_interface name="velocity"/>
@@ -79,6 +79,6 @@
       <joint name="${prefix}joint_6">
         <command_interface name="position">
-          <param name="min">$(-400 * pi / 180)</param>
-          <param name="max">$(400 * pi / 180)</param>
+          <param name="min">${-400 * pi / 180}</param>
+          <param name="max">${400 * pi / 180}</param>
         </command_interface>
         <command_interface name="velocity"/>

File: robot_specific_config/abb_irb120_support/urdf/irb120_3_60_macro.xacro (robot description, xacro)
@@ -7,5 +7,5 @@
       <!-- See note 1 in package.xml about the inertial and mass values -->
       <inertial>
-        <mass value="$(0.006181 * 25 / 0.00912)"/>
+        <mass value="${0.006181 * 25 / 0.00912}"/>
         <origin xyz="-0.041614 0.000184 0.079639"/>
         <inertia ixx="2.461236e-5" ixy="1.712983e-7" ixz="-1.226808e-6" iyy="4.855052e-5" iyz="2.222764e-8" izz="4.663803e-5"/>
@@ -26,5 +26,5 @@
       <!-- See note 1 in package.xml about the inertial and mass values -->
       <inertial>
-        <mass value="$(0.003061 * 25 / 0.00912)"/>
+        <mass value="${0.003061 * 25 / 0.00912}"/>
         <origin xyz="0.000099 -0.000113 -0.051699"/>
         <inertia ixx="1.416505e-5" ixy="1.357926e-8" ixz="2.089039e-8" iyy="1.434604e-5" iyz="-1.885864e-8" izz="1.042534e-5"/>
@@ -45,5 +45,5 @@
       <!-- See note 1 in package.xml about the inertial and mass values -->
       <inertial>
-        <mass value="$(0.003899 * 25 / 0.00912)"/>
+        <mass value="${0.003899 * 25 / 0.00912}"/>
         <origin xyz="0.000770 -0.002098 0.101320"/>
         <inertia ixx="6.007194e-5" ixy="-1.124530e-8" ixz="-5.731156e-8" iyy="4.138268e-5" iyz="4.955519e-7" izz="2.587382e-5"/>
@@ -64,5 +64,5 @@
       <!-- See note 1 in package.xml about the inertial and mass values -->
       <inertial>
-        <mass value="$(0.002939 * 25 / 0.00912)"/>
+        <mass value="${0.002939 * 25 / 0.00912}"/>
         <origin xyz="0.022817 0.001065 0.057957"/>
         <inertia ixx="8.319430e-6" ixy="7.957514e-8" ixz="-1.424078e-6" iyy="1.666783e-5" iyz="1.805283e-7" izz="1.267593e-5"/>
@@ -83,5 +83,5 @@
       <!-- See note 1 in package.xml about the inertial and mass values -->
       <inertial>
-        <mass value="$(0.001324 * 25 / 0.00912)"/>
+        <mass value="${0.001324 * 25 / 0.00912}"/>
         <origin xyz="0.224540 0.000239 0.000433"/>
         <inertia ixx="2.833033e-6" ixy="1.698253e-8" ixz="1.770183e-8" iyy="3.991053e-6" iyz="-1.404654e-8" izz="5.226945e-6"/>
@@ -102,5 +102,5 @@
       <!-- See note 1 in package.xml about the inertial and mass values -->
       <inertial>
-        <mass value="$(0.000548 * 25 / 0.00912)"/>
+        <mass value="${0.000548 * 25 / 0.00912}"/>
         <origin xyz="-0.000811 0.000034 0.000067"/>
         <inertia ixx="4.039701e-7" ixy="-1.305350e-9" ixz="-8.828193e-10" iyy="8.986250e-7" iyz="1.467132e-11" izz="8.222431e-7"/>
@@ -126,5 +126,5 @@
       </inertial> -->
       <inertial>
-        <mass value="$(0.000014 * 25 / 0.00912)"/>
+        <mass value="${0.000014 * 25 / 0.00912}"/>
         <origin xyz="-0.007054 -0.000169 0.000002"/>
         <inertia ixx="2.915416e-9" ixy="7.242353e-12" ixz="1.815316e-13" iyy="1.659334e-9" iyz="-3.419822e-13" izz="1.627338e-9"/>
@@ -150,5 +150,5 @@
       <child link="${prefix}link_1"/>
       <!-- See note 2 in package.xml about effort limits and dynamics values -->
-      <limit effort="1000" lower="$(-165 * pi / 180)" upper="$(165 * pi / 180)" velocity="$(250 * pi / 180)"/>
+      <limit effort="1000" lower="${-165 * pi / 180}" upper="${165 * pi / 180}" velocity="${250 * pi / 180}"/>
       <dynamics damping="50.0" friction="1.0"/>
     </joint>
@@ -159,5 +159,5 @@
       <child link="${prefix}link_2"/>
       <!-- See note 2 in package.xml about effort limits and dynamics values -->
-      <limit effort="1000" lower="$(-110 * pi / 180)" upper="$(110 * pi / 180)" velocity="$(250 * pi / 180)"/>
+      <limit effort="1000" lower="${-110 * pi / 180}" upper="${110 * pi / 180}" velocity="${250 * pi / 180}"/>
       <dynamics damping="50.0" friction="1.0"/>
     </joint>
@@ -168,5 +168,5 @@
       <child link="${prefix}link_3"/>
       <!-- See note 2 in package.xml about effort limits and dynamics values -->
-      <limit effort="1000" lower="$(-110 * pi / 180)" upper="$(70 * pi / 180)" velocity="$(250 * pi / 180)"/>
+      <limit effort="1000" lower="${-110 * pi / 180}" upper="${70 * pi / 180}" velocity="${250 * pi / 180}"/>
       <dynamics damping="10.0" friction="1.0"/>
     </joint>
@@ -177,5 +177,5 @@
       <child link="${prefix}link_4"/>
       <!-- See note 2 in package.xml about effort limits and dynamics values -->
-      <limit effort="1000" lower="$(-160 * pi / 180)" upper="$(160 * pi / 180)" velocity="$(320 * pi / 180)"/>
+      <limit effort="1000" lower="${-160 * pi / 180}" upper="${160 * pi / 180}" velocity="${320 * pi / 180}"/>
       <dynamics damping="5.0" friction="1.0"/>
     </joint>
@@ -186,5 +186,5 @@
       <child link="${prefix}link_5"/>
       <!-- See note 2 in package.xml about effort limits and dynamics values -->
-      <limit effort="1000" lower="$(-120 * pi / 180)" upper="$(120 * pi / 180)" velocity="$(320 * pi / 180)"/>
+      <limit effort="1000" lower="${-120 * pi / 180}" upper="${120 * pi / 180}" velocity="${320 * pi / 180}"/>
       <dynamics damping="2.0" friction="1.0"/>
     </joint>
@@ -195,5 +195,5 @@
       <child link="${prefix}link_6"/>
       <!-- See note 2 in package.xml about effort limits and dynamics values -->
-      <limit effort="1000" lower="$(-400 * pi / 180)" upper="$(400 * pi / 180)" velocity="$(420 * pi / 180)"/>
+      <limit effort="1000" lower="${-400 * pi / 180}" upper="${400 * pi / 180}" velocity="${420 * pi / 180}"/>
       <dynamics damping="1.0" friction="1.0"/>
     </joint>
@@ -216,5 +216,5 @@
     <link name="${prefix}tool0" />
     <joint name="${prefix}link_6-tool0" type="fixed">
-      <origin xyz="0 0 0" rpy="0 ${radians(90)} 0" />
+      <origin xyz="0 0 0" rpy="0 ${radians{90}} 0" />
       <parent link="${prefix}flange" />
       <child link="${prefix}tool0" />

Commit message: Updated xacro expressions to use radians

File: robot_specific_config/abb_irb120_support/urdf/irb120.ros2_control.xacro (robot description, xacro)
@@ -24,6 +24,6 @@
       <joint name="${prefix}joint_1">
         <command_interface name="position">
-          <param name="min">${-165 * pi / 180}</param>
-          <param name="max">${165 * pi / 180}</param>
+          <param name="min">${radians(-165)}</param>
+          <param name="max">${radians(165)}</param>
         </command_interface>
         <command_interface name="velocity"/>
@@ -35,6 +35,6 @@
       <joint name="${prefix}joint_2">
         <command_interface name="position">
-          <param name="min">${-110 * pi / 180}</param>
-          <param name="max">${110 * pi / 180}</param>
+          <param name="min">${radians(-110)}</param>
+          <param name="max">${radians(110)}</param>
         </command_interface>
         <command_interface name="velocity"/>
@@ -46,6 +46,6 @@
       <joint name="${prefix}joint_3">
         <command_interface name="position">
-          <param name="min">${-110 * pi / 180}</param>
-          <param name="max">${70 * pi / 180}</param>
+          <param name="min">${radians(-110)}</param>
+          <param name="max">${radians(70)}</param>
         </command_interface>
         <command_interface name="velocity"/>
@@ -57,6 +57,6 @@
       <joint name="${prefix}joint_4">
         <command_interface name="position">
-          <param name="min">${-160 * pi / 180}</param>
-          <param name="max">${160 * pi / 180}</param>
+          <param name="min">${radians(-160)}</param>
+          <param name="max">${radians(160)}</param>
         </command_interface>
         <command_interface name="velocity"/>
@@ -68,6 +68,6 @@
       <joint name="${prefix}joint_5">
         <command_interface name="position">
-          <param name="min">${-120 * pi / 180}</param>
-          <param name="max">${120 * pi / 180}</param>
+          <param name="min">${radians(-120)}</param>
+          <param name="max">${radians(120)}</param>
         </command_interface>
         <command_interface name="velocity"/>
@@ -79,6 +79,6 @@
       <joint name="${prefix}joint_6">
         <command_interface name="position">
-          <param name="min">${-400 * pi / 180}</param>
-          <param name="max">${400 * pi / 180}</param>
+          <param name="min">${radians(-400)}</param>
+          <param name="max">${radians(400)}</param>
         </command_interface>
         <command_interface name="velocity"/>

File: robot_specific_config/abb_irb120_support/urdf/irb120_3_60_macro.xacro (robot description, xacro)
@@ -150,5 +150,5 @@
       <child link="${prefix}link_1"/>
       <!-- See note 2 in package.xml about effort limits and dynamics values -->
-      <limit effort="1000" lower="${-165 * pi / 180}" upper="${165 * pi / 180}" velocity="${250 * pi / 180}"/>
+      <limit effort="1000" lower="${radians(-165)}" upper="${radians(165)}" velocity="${radians(250)}"/>
       <dynamics damping="50.0" friction="1.0"/>
     </joint>
@@ -159,5 +159,5 @@
       <child link="${prefix}link_2"/>
       <!-- See note 2 in package.xml about effort limits and dynamics values -->
-      <limit effort="1000" lower="${-110 * pi / 180}" upper="${110 * pi / 180}" velocity="${250 * pi / 180}"/>
+      <limit effort="1000" lower="${radians(-110)}" upper="${radians(110)}" velocity="${radians(250)}"/>
       <dynamics damping="50.0" friction="1.0"/>
     </joint>
@@ -168,5 +168,5 @@
       <child link="${prefix}link_3"/>
       <!-- See note 2 in package.xml about effort limits and dynamics values -->
-      <limit effort="1000" lower="${-110 * pi / 180}" upper="${70 * pi / 180}" velocity="${250 * pi / 180}"/>
+      <limit effort="1000" lower="${radians(-110)}" upper="${radians(70)}" velocity="${radians(250)}"/>
       <dynamics damping="10.0" friction="1.0"/>
     </joint>
@@ -177,5 +177,5 @@
       <child link="${prefix}link_4"/>
       <!-- See note 2 in package.xml about effort limits and dynamics values -->
-      <limit effort="1000" lower="${-160 * pi / 180}" upper="${160 * pi / 180}" velocity="${320 * pi / 180}"/>
+      <limit effort="1000" lower="${radians(-160)}" upper="${radians(160)}" velocity="${radians(320)}"/>
       <dynamics damping="5.0" friction="1.0"/>
     </joint>
@@ -186,5 +186,5 @@
       <child link="${prefix}link_5"/>
       <!-- See note 2 in package.xml about effort limits and dynamics values -->
-      <limit effort="1000" lower="${-120 * pi / 180}" upper="${120 * pi / 180}" velocity="${320 * pi / 180}"/>
+      <limit effort="1000" lower="${radians(-120)}" upper="${radians(120)}" velocity="${radians(320)}"/>
       <dynamics damping="2.0" friction="1.0"/>
     </joint>
@@ -195,5 +195,5 @@
       <child link="${prefix}link_6"/>
       <!-- See note 2 in package.xml about effort limits and dynamics values -->
-      <limit effort="1000" lower="${-400 * pi / 180}" upper="${400 * pi / 180}" velocity="${420 * pi / 180}"/>
+      <limit effort="1000" lower="${radians(-400)}" upper="${radians(400)}" velocity="${radians(420)}"/>
       <dynamics damping="1.0" friction="1.0"/>
     </joint>
@@ -216,5 +216,5 @@
     <link name="${prefix}tool0" />
     <joint name="${prefix}link_6-tool0" type="fixed">
-      <origin xyz="0 0 0" rpy="0 ${radians{90}} 0" />
+      <origin xyz="0 0 0" rpy="0 ${radians(90)} 0" />
       <parent link="${prefix}flange" />
       <child link="${prefix}tool0" />
